File: rtl8723bs-tryout.sch (KiCad schematic (older format))
At the start: 13 parts

Commit message: update footprint,
Parts:
- AE1: renamed from AE?; footprint (none) -> footprint-lib:rainsun-AN9520
- J1: renamed from J?; value Conn_01x06 -> SDC_DEBUG; footprint (none) -> Connector_PinHeader_2.54mm:PinHeader_1x06_P2.54mm_Vertical
- J2: renamed from J?; value Conn_01x03 -> UART_DEBUG; footprint (none) -> Connector_PinHeader_2.54mm:PinHeader_1x03_P2.54mm_Vertical
- U8: renamed from U?; footprint (none) -> footprint-lib:RL-SM02BD(RTL8723BS)
- gave numbers to parts that had none: 9
Changed lines of the file:
@@
 $EndBitmap
 $Comp
-L taobao-components:RTL8723BS U?
+L taobao-components:RTL8723BS U8
 U 1 1 5E58D194
 P 4250 1950
-F 0 "U?" H 4200 3165 50  0000 C CNN
+F 0 "U8" H 4200 3165 50  0000 C CNN
 F 1 "RTL8723BS" H 4200 3074 50  0000 C CNN
-F 2 "" H 4250 1950 50  0001 C CNN
+F 2 "footprint-lib:RL-SM02BD(RTL8723BS)" H 4250 1950 50  0001 C CNN
 F 3 "" H 4250 1950 50  0001 C CNN
 	1    4250 1950
@@
 $EndComp
 $Comp
-L Connector_Generic:Conn_01x03 J?
+L Connector_Generic:Conn_01x03 J2
 U 1 1 5E58EF3B
 P 6050 1100
-F 0 "J?" H 5968 775 50  0000 C CNN
-F 1 "Conn_01x03" H 5968 866 50  0000 C CNN
-F 2 "" H 6050 1100 50  0001 C CNN
+F 0 "J2" H 5968 775 50  0000 C CNN
+F 1 "UART_DEBUG" H 5968 866 50  0000 C CNN
+F 2 "Connector_PinHeader_2.54mm:PinHeader_1x03_P2.54mm_Vertical" H 6050 1100 50  0001 C CNN
 F 3 "~" H 6050 1100 50  0001 C CNN
 	1    6050 1100
@@
 	4950 1200 5850 1200
 $Comp
-L power:GND #PWR?
+L power:GND #PWR09
 U 1 1 5E590680
 P 5650 1300
-F 0 "#PWR?" H 5650 1050 50  0001 C CNN
+F 0 "#PWR09" H 5650 1050 50  0001 C CNN
 F 1 "GND" V 5655 1172 50  0000 R CNN
 F 2 "" H 5650 1300 50  0001 C CNN
@@
 	5650 1300 4950 1300
 $Comp
-L power:GND #PWR?
+L power:GND #PWR010
 U 1 1 5E590CE9
 P 5650 1800
-F 0 "#PWR?" H 5650 1550 50  0001 C CNN
+F 0 "#PWR010" H 5650 1550 50  0001 C CNN
 F 1 "GND" V 5655 1672 50  0000 R CNN
 F 2 "" H 5650 1800 50  0001 C CNN
@@
 	5650 1800 4950 1800
 $Comp
-L power:GND #PWR?
+L power:GND #PWR011
 U 1 1 5E591FEA
 P 5650 2100
-F 0 "#PWR?" H 5650 1850 50  0001 C CNN
+F 0 "#PWR011" H 5650 1850 50  0001 C CNN
 F 1 "GND" V 5655 1972 50  0000 R CNN
 F 2 "" H 5650 2100 50  0001 C CNN
@@
 	5650 2100 4950 2100
 $Comp
-L power:GND #PWR?
+L power:GND #PWR012
 U 1 1 5E592859
 P 5650 2300
-F 0 "#PWR?" H 5650 2050 50  0001 C CNN
+F 0 "#PWR012" H 5650 2050 50  0001 C CNN
 F 1 "GND" V 5655 2172 50  0000 R CNN
 F 2 "" H 5650 2300 50  0001 C CNN
@@
 	5650 2300 4950 2300
 $Comp
-L customized_power:+3V3 #PWR?
+L customized_power:+3V3 #PWR014
 U 1 1 5E5934CE
 P 5900 3100
-F 0 "#PWR?" H 5900 2950 50  0001 C CNN
+F 0 "#PWR014" H 5900 2950 50  0001 C CNN
 F 1 "+3V3" V 5915 3228 50  0000 L CNN
 F 2 "" H 5900 3100 50  0001 C CNN
@@
 $EndComp
 $Comp
-L sz_jlc_resistor:10KΩ,(1002),±1%,0603,C25804 U?
+L sz_jlc_resistor:10KΩ,(1002),±1%,0603,C25804 U10
 U 1 1 5E5944D4
 P 5400 3100
-F 0 "U?" V 5204 3100 50  0000 C CNN
+F 0 "U10" V 5204 3100 50  0000 C CNN
 F 1 "10KΩ,(1002),±1%,0603,C25804" V 5295 3100 50  0000 C CNN
 F 2 "w_smd_resistors:r_0603" H 5400 2100 50  0001 C CNN
@@
 	5500 3100 5900 3100
 $Comp
-L customized_power:+3V3 #PWR?
+L customized_power:+3V3 #PWR013
 U 1 1 5E595D9D
 P 5900 2000
-F 0 "#PWR?" H 5900 1850 50  0001 C CNN
+F 0 "#PWR013" H 5900 1850 50  0001 C CNN
 F 1 "+3V3" V 5915 2128 50  0000 L CNN
 F 2 "" H 5900 2000 50  0001 C CNN
@@
 	5500 2000 5900 2000
 $Comp
-L Connector_Generic:Conn_01x06 J?
+L Connector_Generic:Conn_01x06 J1
 U 1 1 5E598990
 P 3500 4100
-F 0 "J?" H 3580 4092 50  0000 L CNN
-F 1 "Conn_01x06" H 3580 4001 50  0000 L CNN
-F 2 "" H 3500 4100 50  0001 C CNN
+F 0 "J1" H 3580 4092 50  0000 L CNN
+F 1 "SDC_DEBUG" H 3580 4001 50  0000 L CNN
+F 2 "Connector_PinHeader_2.54mm:PinHeader_1x06_P2.54mm_Vertical" H 3500 4100 50  0001 C CNN
 F 3 "~" H 3500 4100 50  0001 C CNN
 	1    3500 4100
@@
 	2550 4400 3300 4400
 $Comp
-L sz_jlc_resistor:47KΩ,(4702),±1%,0603,C25819 U?
+L sz_jlc_resistor:47KΩ,(4702),±1%,0603,C25819 U1
 U 1 1 5E5A1C63
 P 1350 3950
-F 0 "U?" V 1154 3950 50  0000 C CNN
+F 0 "U1" V 1154 3950 50  0000 C CNN
 F 1 "47KΩ,(4702),±1%,0603,C25819" V 1245 3950 50  0000 C CNN
 F 2 "w_smd_resistors:r_0603" H 1350 2950 50  0001 C CNN
@@
 $EndComp
 $Comp
-L customized_power:+3V3 #PWR?
+L customized_power:+3V3 #PWR01
 U 1 1 5E5A285C
 P 900 3650
-F 0 "#PWR?" H 900 3500 50  0001 C CNN
+F 0 "#PWR01" H 900 3500 50  0001 C CNN
 F 1 "+3V3" H 915 3823 50  0000 C CNN
 F 2 "" H 900 3650 50  0001 C CNN
@@
 $EndComp
 $Comp
-L sz_jlc_resistor:47KΩ,(4702),±1%,0603,C25819 U?
+L sz_jlc_resistor:47KΩ,(4702),±1%,0603,C25819 U2
 U 1 1 5E5A2C30
 P 1350 4100
-F 0 "U?" V 1154 4100 50  0000 C CNN
+F 0 "U2" V 1154 4100 50  0000 C CNN
 F 1 "47KΩ,(4702),±1%,0603,C25819" V 1245 4100 50  0000 C CNN
 F 2 "w_smd_resistors:r_0603" H 1350 3100 50  0001 C CNN
@@
 $EndComp
 $Comp
-L sz_jlc_resistor:47KΩ,(4702),±1%,0603,C25819 U?
+L sz_jlc_resistor:47KΩ,(4702),±1%,0603,C25819 U3
 U 1 1 5E5A2DF7
 P 1350 4250
-F 0 "U?" V 1154 4250 50  0000 C CNN
+F 0 "U3" V 1154 4250 50  0000 C CNN
 F 1 "47KΩ,(4702),±1%,0603,C25819" V 1245 4250 50  0000 C CNN
 F 2 "w_smd_resistors:r_0603" H 1350 3250 50  0001 C CNN
@@
 $EndComp
 $Comp
-L sz_jlc_resistor:47KΩ,(4702),±1%,0603,C25819 U?
+L sz_jlc_resistor:47KΩ,(4702),±1%,0603,C25819 U4
 U 1 1 5E5A302E
 P 1350 4400
-F 0 "U?" V 1154 4400 50  0000 C CNN
+F 0 "U4" V 1154 4400 50  0000 C CNN
 F 1 "47KΩ,(4702),±1%,0603,C25819" V 1245 4400 50  0000 C CNN
 F 2 "w_smd_resistors:r_0603" H 1350 3400 50  0001 C CNN
@@
 $EndComp
 $Comp
-L sz_jlc_resistor:47KΩ,(4702),±1%,0603,C25819 U?
+L sz_jlc_resistor:47KΩ,(4702),±1%,0603,C25819 U5
 U 1 1 5E5A31FD
 P 1350 4550
-F 0 "U?" V 1454 4550 50  0000 C CNN
+F 0 "U5" V 1454 4550 50  0000 C CNN
 F 1 "47KΩ,(4702),±1%,0603,C25819" V 1545 4550 50  0000 C CNN
 F 2 "w_smd_resistors:r_0603" H 1350 3550 50  0001 C CNN
@@
 	2200 4550 1450 4550
 $Comp
-L power:GND #PWR?
+L power:GND #PWR06
 U 1 1 5E5AC216
 P 2750 1000
-F 0 "#PWR?" H 2750 750 50  0001 C CNN
+F 0 "#PWR06" H 2750 750 50  0001 C CNN
 F 1 "GND" V 2755 872 50  0000 R CNN
 F 2 "" H 2750 1000 50  0001 C CNN
@@
 	2750 1000 3450 1000
 $Comp
-L power:GND #PWR?
+L power:GND #PWR07
 U 1 1 5E5AF201
 P 2750 1200
-F 0 "#PWR?" H 2750 950 50  0001 C CNN
+F 0 "#PWR07" H 2750 950 50  0001 C CNN
 F 1 "GND" V 2755 1072 50  0000 R CNN
 F 2 "" H 2750 1200 50  0001 C CNN
@@
 BT_H_WK
 $Comp
-L sz_jlc_resistor:100KΩ,(1003),±1%,0603,C25803 U?
+L sz_jlc_resistor:100KΩ,(1003),±1%,0603,C25803 U9
 U 1 1 5E5B14A7
 P 5400 2000
-F 0 "U?" V 5204 2000 50  0000 C CNN
+F 0 "U9" V 5204 2000 50  0000 C CNN
 F 1 "100KΩ,(1003),±1%,0603,C25803" V 5295 2000 50  0000 C CNN
 F 2 "w_smd_resistors:r_0603" H 5400 1000 50  0001 C CNN
@@
 	3000 1600 3450 1600
 $Comp
-L customized_power:+3V3 #PWR?
+L customized_power:+3V3 #PWR03
 U 1 1 5E5B375D
 P 2700 1800
-F 0 "#PWR?" H 2700 1650 50  0001 C CNN
+F 0 "#PWR03" H 2700 1650 50  0001 C CNN
 F 1 "+3V3" V 2715 1928 50  0000 L CNN
 F 2 "" H 2700 1800 50  0001 C CNN
@@
 	3450 1800 2700 1800
 $Comp
-L customized_power:+3V3 #PWR?
+L customized_power:+3V3 #PWR04
 U 1 1 5E5B4D67
 P 2700 2100
-F 0 "#PWR?" H 2700 1950 50  0001 C CNN
+F 0 "#PWR04" H 2700 1950 50  0001 C CNN
 F 1 "+3V3" V 2715 2228 50  0000 L CNN
 F 2 "" H 2700 2100 50  0001 C CNN
@@
 $EndComp
 $Comp
-L sz_jlc_resistor:100KΩ,(1003),±1%,0603,C25803 U?
+L sz_jlc_resistor:100KΩ,(1003),±1%,0603,C25803 U7
 U 1 1 5E5B5081
 P 3100 2100
-F 0 "U?" V 2904 2100 50  0000 C CNN
+F 0 "U7" V 2904 2100 50  0000 C CNN
 F 1 "100KΩ,(1003),±1%,0603,C25803" V 2995 2100 50  0000 C CNN
 F 2 "w_smd_resistors:r_0603" H 3100 1100 50  0001 C CNN
@@
 	3200 2100 3450 2100
 $Comp
-L power:GND #PWR?
+L power:GND #PWR08
 U 1 1 5E5B8433
 P 3200 2900
-F 0 "#PWR?" H 3200 2650 50  0001 C CNN
+F 0 "#PWR08" H 3200 2650 50  0001 C CNN
 F 1 "GND" V 3205 2772 50  0000 R CNN
 F 2 "" H 3200 2900 50  0001 C CNN
@@
 	3200 2900 3450 2900
 $Comp
-L customized_power:+3V3 #PWR?
+L customized_power:+3V3 #PWR05
 U 1 1 5E5C0D12
 P 2700 3100
-F 0 "#PWR?" H 2700 2950 50  0001 C CNN
+F 0 "#PWR05" H 2700 2950 50  0001 C CNN
 F 1 "+3V3" V 2715 3228 50  0000 L CNN
 F 2 "" H 2700 3100 50  0001 C CNN
@@
 	2700 2800 3450 2800
 $Comp
-L Device:Antenna_Shield AE?
+L Device:Antenna_Shield AE1
 U 1 1 5E5DDE20
 P 1250 750
-F 0 "AE?" H 1394 789 50  0000 L CNN
+F 0 "AE1" H 1394 789 50  0000 L CNN
 F 1 "Antenna_Shield" H 1394 698 50  0000 L CNN
-F 2 "" H 1250 850 50  0001 C CNN
+F 2 "footprint-lib:rainsun-AN9520" H 1250 850 50  0001 C CNN
 F 3 "~" H 1250 850 50  0001 C CNN
 	1    1250 750
@@
 $EndComp
 $Comp
-L power:GND #PWR?
+L power:GND #PWR02
 U 1 1 5E5DE64D
 P 1350 1300
-F 0 "#PWR?" H 1350 1050 50  0001 C CNN
+F 0 "#PWR02" H 1350 1050 50  0001 C CNN
 F 1 "GND" H 1355 1127 50  0000 C CNN
 F 2 "" H 1350 1300 50  0001 C CNN
@@
 	1350 950  1350 1300
 $Comp
-L sz_jlc_capacitor:33pF,(330),±5%,50V,C0G,0603,C1663 U?
+L sz_jlc_capacitor:33pF,(330),±5%,50V,C0G,0603,C1663 U6
 U 1 1 5E5E0713
 P 1850 1100
-F 0 "U?" V 1621 1100 50  0000 C CNN
+F 0 "U6" V 1621 1100 50  0000 C CNN
 F 1 "33pF,(330),±5%,50V,C0G,0603,C1663" V 1712 1100 50  0000 C CNN
 F 2 "w_smd_cap:c_0603" H 1850 100 50  0001 C CNN
